Commit message: finished node for ndof-it is actually only 6dof

File: urdf/dynamixel_wrist.xacro (robot description, xacro)
@@ -31,10 +31,11 @@
       origin_rpy="0 0 0"
       color_rgba="0.10 0.10 0.80 1.0" />
-    <xacro:dxlPROp_wrist_joint
+    <xacro:dxlPROp_cont_wrist_joint
       active_name="${prefix}_dxl_${roll1}_sta__${prefix}_dxl_${roll1}_mov"
       active_origin_rpy="0 0 0"
       active_origin_xyz="0 0.009 0"
       active_parent="${prefix}_dxl_${roll1}_sta"
-      active_child="${prefix}_conn_${pitch}"/>
+      active_child="${prefix}_conn_${pitch}"
+      is_continuous="true"/>
     <xacro:active_a110_connector
       name="${prefix}_conn_${pitch}"
@@ -80,10 +81,11 @@
       origin_rpy="0 0 0"
       color_rgba="0.10 0.80 0.10 1.0" />
-    <xacro:dxlPROp_wrist_joint
+    <xacro:dxlPROp_cont_wrist_joint
       active_name="${prefix}_dxl_${roll2}_sta__${child_link}"
       active_origin_rpy="0 0 0"
       active_origin_xyz="0 0.009 0"
       active_parent="${prefix}_dxl_${roll2}_sta"
-      active_child="${child_link}"/>
+      active_child="${child_link}"
+      is_continuous="true"/>
   </xacro:macro>
 </robot>

File: urdf/modules.xacro (robot description, xacro)
@@ -353,4 +353,28 @@
     </joint>
 </xacro:macro>
+<!-- Synthetic joint parameters -->
+<xacro:macro name="dxlPROp_cont_wrist_joint"
+             params="active_name
+                     active_origin_rpy
+                     active_origin_xyz
+                     active_parent
+                     active_child
+                     is_continuous:=false">
+  <joint name="${active_name}"
+         type="${'continuous' if is_continuous else 'revolute'}">
+    <origin rpy="${active_origin_rpy}" xyz="${active_origin_xyz}" />
+    <parent link="${active_parent}" />
+    <child link="${active_child}" />
+    <axis xyz="0 1 0"/>
+    <!-- Limits only for revolute joints -->
+    <xacro:unless value="${is_continuous}">
+      <limit effort="55"
+             lower="-2"
+             upper="2"
+             velocity="4.0841"/>
+    </xacro:unless>
+    <dynamics damping="10.0" friction="10.0"/>
+  </joint>
+</xacro:macro>
 <!-- FORCE SENSOR -->
 <xacro:macro name="force_sensor" params="name">
@@ -381,29 +405,40 @@
 </xacro:macro>
 <!-- FORCE SENSOR CIRC ASSEMBLY - 6DOF ONLY [ASSEMBLED AFTER WRIST] -->
-<xacro:macro name="force_sensor_circ" params="name">
-	<link name="${name}">
-	    <inertial>
-	      <origin rpy="0 0 0" xyz="0 0 0"/>
-	      <mass value ="0.250" />
-	      <inertia ixx="5.294e-005" ixy="-2.2e-007" ixz="-3.787e-008" iyy="5.233e-005" iyz="-2.827e-008" izz="4.192e-005"/>
-	    </inertial>
-	    <visual>
-	      <origin rpy="-1.5708 -3.1416 0" xyz="0 0.0725 0"/>
-	      <geometry>
-	        <mesh filename="package://smm_synthesis/meshes/massage_circ_assembly.stl" scale="0.001 0.001 0.001"/>
-	      </geometry>
-	      <material name="edward">
-	        <!-- Color Pick: http://www.flatuicolorpicker.com/grey-rgba-color-model/ -->
-	        <color rgba="0.6705 0.7098 0.7098 1"/>
-	      </material>
-	    </visual>
-	<!-- Added on [16-2-24]. Checked visually by executing: $ roslaunch smm_synthesis smm_ros_gazebo.launch -->
-    	<collision>
-    		<origin rpy="1.5708 0 0" xyz="0 0.015 0" />
-      		<geometry>
-        		  <cylinder length="0.035" radius="0.03"/>
-      		</geometry>
-    	</collision>
-	</link>
+<xacro:macro name="force_sensor_circ" params="name meas_frame_name">
+  <!-- Physical sensor link -->
+  <link name="${name}">
+    <inertial>
+      <origin rpy="0 0 0" xyz="0 0 0"/>
+      <mass value="0.250"/>
+      <inertia ixx="5.294e-005" ixy="-2.2e-007" ixz="-3.787e-008"
+               iyy="5.233e-005" iyz="-2.827e-008" izz="4.192e-005"/>
+    </inertial>
+    <visual>
+      <origin rpy="-1.5708 -3.1416 0" xyz="0 0.0725 0"/>
+      <geometry>
+        <mesh filename="package://smm_synthesis/meshes/massage_circ_assembly.stl"
+              scale="0.001 0.001 0.001"/>
+      </geometry>
+      <material name="edward">
+        <color rgba="0.6705 0.7098 0.7098 1"/>
+      </material>
+    </visual>
+    <collision>
+      <origin rpy="1.5708 0 0" xyz="0 0.015 0"/>
+      <geometry>
+        <cylinder length="0.035" radius="0.03"/>
+      </geometry>
+    </collision>
+  </link>
+  <!-- Measurement frame (massless, invisible) -->
+  <link name="${meas_frame_name}"/>
+  <!-- Fixed joint defining measurement frame orientation -->
+  <joint name="${name}_meas_frame_joint" type="fixed">
+    <parent link="${name}"/>
+    <child link="${meas_frame_name}"/>
+    <!-- Here we define the sensor coordinate frame - aligned with datasheet axes !!! -->
+    <origin xyz="0 0.02 0"
+            rpy="1.5708 1.5708 0"/>
+  </joint>
 </xacro:macro>
 <!-- END-EFFECTOR-TOOL/MASSAGE-TOOL-XACRO-VISUALS-->
@@ -515,3 +550,39 @@
 	</link>
 </xacro:macro>
+<!-- MASSAGE-TOOL-STL CIRC ASSEMBLY - 6DOF ONLY [ASSEMBLED AFTER WRIST] -->
+<xacro:macro name="massage_tool_stl_6dof" params="name tcp_frame_name tcp_xyz:='0 0 0' tcp_rpy:='0 0 0'">
+  <!-- Physical tool link -->
+  <link name="${name}">
+    <inertial>
+      <origin rpy="0 0 0" xyz="0 0 0"/>
+      <mass value="0.250" />
+      <inertia ixx="6.414e-005" ixy="0" ixz="0"
+               iyy="6.414e-005" iyz="0" izz="4.986e-005"/>
+    </inertial>
+    <visual>
+      <origin rpy="0 0 0" xyz="0 0 0"/>
+      <geometry>
+        <mesh filename="package://smm_synthesis/meshes/massage_tool_circ_assembly.stl"
+              scale="0.001 0.001 0.001"/>
+      </geometry>
+      <material name="Porcelain">
+        <color rgba="0.9254 0.9412 0.9413 1"/>
+      </material>
+    </visual>
+    <collision>
+      <origin rpy="0 0 0" xyz="0 0 0.02" />
+      <geometry>
+        <sphere radius="0.03"/>
+      </geometry>
+    </collision>
+  </link>
+  <!-- TCP frame: massless, collision-less -->
+  <link name="${tcp_frame_name}"/>
+  <!-- Fixed joint defining TCP pose relative to the tool link -->
+  <joint name="${name}__tcp" type="fixed">
+    <parent link="${name}"/>
+    <child link="${tcp_frame_name}"/>
+    <origin xyz="${tcp_xyz}" rpy="${tcp_rpy}"/>
+  </joint>
+</xacro:macro>
 </robot>

File: urdf/smm_structure_anatomy_assembly_6dof.xacro (robot description, xacro)
@@ -379,4 +379,5 @@
 <!-- SPHERICAL WRIST COMPOSED OF DYNAMIXELS -->
 <xacro:property name="force_sensor" value="force_sensor_circ" />
+<xacro:property name="force_sensor_meas_frame" value="force_sensor_meas" />
 <xacro:dynamixel_wrist
 parent_link="${last_body_assembled}"
@@ -386,14 +387,18 @@
 origin_rpy="0 0 0" />
 <!-- FORCE SENSOR -->
-<xacro:force_sensor_circ name="${force_sensor}"/>
+<xacro:force_sensor_circ name="${force_sensor}" meas_frame_name="${force_sensor_meas_frame}"/>
 <!-- [1-3-24] Enable only 1 option for END-EFFECTOR-->
 <!-- Default option: massage_tool_is_stl = true  -->
 <xacro:if value="${massage_tool_is_stl}">
-	<joint name="${force_sensor}__massage_tool" type="fixed">
-		<origin rpy="-1.5708 0 0" xyz="0 0.060 0"/>
-		<parent link="${force_sensor}"/>
+	<joint name="${force_sensor_meas_frame}__massage_tool" type="fixed">
+		<origin rpy="0 -3.1416 0" xyz="0 0 -0.040"/>
+		<parent link="${force_sensor_meas_frame}"/>
 		<child link="${massage_tool_stl}"/>
 	</joint>
-	<xacro:massage_tool_stl_6dof name="${massage_tool_stl}" />
+  <xacro:massage_tool_stl_6dof
+  name="${massage_tool_stl}"
+  tcp_frame_name="tcp"
+  tcp_xyz="0 0 0.045"
+  tcp_rpy="0 0 0"/>
   <gazebo reference="${massage_tool_stl}">
     <material>Gazebo/Orange</material>
