Commit message: restructured for user-friendly and interoperability upgrade

File: urdf/3dof/smm_structure_anatomy_assembly_3dof.xacro (robot description, xacro)
@@ -21,10 +21,12 @@
 <xacro:include filename="$(find smm_synthesis)/urdf/transmissions.xacro" />
 <!-- I.3	INCLUDE YAML WITH FIXED CONNECTIVITY/ASSEMBLY PARAMETERS-->
-<xacro:property name="connectivity_yaml" value="$(find smm_synthesis)/config/yaml/connectivity.yaml" />
+<xacro:property name="connectivity_yaml" value="$(find smm_synthesis)/config/yaml/3dof/connectivity_3dof.yaml" />
 <!-- I.4	INCLUDE YAML WITH DESIRED STRUCTURE/ANATOMY PARAMETERS-->
 <!-- <xacro:property name="pseudo_angles_definitions" value="$(find smm_synthesis)/config/yaml/pseudo_angles.yaml" /> --> <!-- DEPRECATED -->
 <!-- <xacro:property name="structure_string_definitions" value="$(find smm_synthesis)/config/yaml/structure_string.yaml" /> -->  <!-- DEPRECATED -->
 <!-- <xacro:property name="ovidius_assembly_parameters_file" value="$(find smm_synthesis)/config/yaml/smm_assembly_parameters.yaml" /> -->  <!-- DEPRECATED -->
-<xacro:property name="assembly_yaml" value="$(find smm_synthesis)/config/yaml/assembly.yaml" /> <!-- [26-4-25] MERGES YAML FILES: structure_string, smm_assembly_parameters, pseudo_angles -->
+<!-- [26-04-25] NEW ASSEMBLY TEMPLATE CREATED: MERGES YAML FILES: structure_string, smm_assembly_parameters, pseudo_angles -->
+<!-- [07-02-26] CAHNGED FOLDER STRUCTURE IN ORDER TO BE USER-FRIENDLY FOR MULTIPLE DOF's-->
+<xacro:property name="assembly_yaml" value="$(find smm_synthesis)/config/yaml/3dof/assembly_3dof.yaml" />
 <!-- VIRTUAL JOINT-->
 <xacro:property name="virtual_joint" value="${xacro.load_yaml(connectivity_yaml)}"/>

File: urdf/6dof/smm_structure_anatomy_assembly_6dof.xacro (robot description, xacro)
@@ -28,7 +28,7 @@
 <xacro:include filename="$(find smm_synthesis)/urdf/dynamixel_wrist.xacro" />
 <!-- I.2.1	INCLUDE YAML WITH FIXED CONNECTIVITY/ASSEMBLY PARAMETERS-->
-<xacro:property name="connectivity_yaml" value="$(find smm_synthesis)/config/yaml/connectivity_6dof.yaml" />
+<xacro:property name="connectivity_yaml" value="$(find smm_synthesis)/config/yaml/6dof/connectivity_6dof.yaml" />
 <!-- I.2.2	INCLUDE YAML WITH DESIRED STRUCTURE/ANATOMY PARAMETERS-->
-<xacro:property name="assembly_yaml" value="$(find smm_synthesis)/config/yaml/assembly_6dof.yaml" />
+<xacro:property name="assembly_yaml" value="$(find smm_synthesis)/config/yaml/6dof/assembly_6dof.yaml" />
 <!-- VIRTUAL JOINT-->
 <xacro:property name="virtual_joint" value="${xacro.load_yaml(connectivity_yaml)}"/>

Commit message: debug ok, exports for 6dof

File: urdf/3dof/smm_structure_anatomy_assembly_3dof.xacro (robot description, xacro)
@@ -338,5 +338,15 @@
 		<child link="${massage_tool_stl}"/>
 	</joint>
-	<xacro:massage_tool_stl name="${massage_tool_stl}" />
+  <!-- [10-2-2026] Replaced old macro for massage tool frame with a new (6dof based)-->
+	<!-- <xacro:massage_tool_stl name="${massage_tool_stl}" />
+  <gazebo reference="${massage_tool_stl}">
+    <material>Gazebo/Orange</material>
+  </gazebo> -->
+    <!-- New macro: tool + tcp -->
+  <xacro:massage_tool_stl_3dof
+    name="${massage_tool_stl}"
+    tcp_frame_name="tcp"
+    tcp_xyz="0 0 0.045"
+    tcp_rpy="0 0 0"/>
   <gazebo reference="${massage_tool_stl}">
     <material>Gazebo/Orange</material>

File: urdf/modules.xacro (robot description, xacro)
@@ -523,4 +523,44 @@
 	</link>
 </xacro:macro>
+<!-- MASSAGE-TOOL-STL + TCP FRAME (3DOF VERSION) -->
+<xacro:macro name="massage_tool_stl_3dof"
+             params="name tcp_frame_name tcp_xyz:='0 0 0.045' tcp_rpy:='0 0 0'">
+  <!-- Physical tool link: same geometry / inertia as massage_tool_stl -->
+  <link name="${name}">
+    <inertial>
+      <!-- from massage_tool_stl -->
+      <origin rpy="0 0 0" xyz="0 0 0.0378"/>
+      <mass value ="0.211" />
+      <inertia ixx="6.414e-005" ixy="0" ixz="0"
+               iyy="6.414e-005" iyz="0" izz="4.986e-005"/>
+    </inertial>
+    <visual>
+      <!-- from massage_tool_stl -->
+      <origin rpy="0 0 0" xyz="0 0 0.020"/>
+      <geometry>
+        <mesh filename="package://smm_synthesis/meshes/massage_tool.stl"
+              scale="0.001 0.001 0.001"/>
+      </geometry>
+      <material name="Porcelain">
+        <color rgba="0.9254 0.9412 0.9413 1"/>
+      </material>
+    </visual>
+    <collision>
+      <!-- from massage_tool_stl -->
+      <origin rpy="0 0 0" xyz="0 0 0.040" />
+      <geometry>
+        <sphere radius="0.025"/>
+      </geometry>
+    </collision>
+  </link>
+  <!-- TCP frame: massless, collisionless -->
+  <link name="${tcp_frame_name}"/>
+  <!-- Fixed joint defining TCP pose relative to the tool link -->
+  <joint name="${name}__tcp" type="fixed">
+    <parent link="${name}"/>
+    <child link="${tcp_frame_name}"/>
+    <origin xyz="${tcp_xyz}" rpy="${tcp_rpy}"/>
+  </joint>
+</xacro:macro>
 <!-- MASSAGE-TOOL-STL CIRC ASSEMBLY - 6DOF ONLY [ASSEMBLED AFTER WRIST] -->
 <xacro:macro name="massage_tool_stl_6dof" params="name">
